File: electrical/shrew.brd (EAGLE design)
At the start: 18 x 30 mm, 20 parts, among them U1 ESP32-PICO-D4, U2 SX1280IMLTRT, U3 DRV8231DSGR, U4 DRV8231DSGR, Y1 OSCILLATOR-TG2016SMN

Commit message: wip, before splitting board into modules
Parts:
- added C10, C11: (no value), shrew-common:0402-CAP
- added C12, C13, C14, C15, C16, C18, C19, C20: (no value), shrew-common:0805
- added C17: 100n, shrew-common:0402-CAP
- added FIDUCIAL1, FIDUCIAL2: FIDUCIAL-1MM-2MM, shrew-core:FIDUCIAL-1MM-2MM
- added IC1: (no value), shrew-common:SOT223
- added JP1: (no value), shrew-common:1X03
- added JP2: (no value), shrew-common:1X04
- added JP3, JP4: (no value), shrew-common:1X07-2MM-TH
- added LED1: SK6812-EC20, shrew-core:SK6812-EC20
- added R2: 10K, shrew-common:0402-RES
- added R3: 470K, shrew-common:0402-RES
- added TOOLING1, TOOLING2, TOOLING3: TOOLING-HOLE, shrew-core:TOOLING-HOLE
- added U5: DRV8244HQRYJRQ1, shrew-core:RYJ0016A-MFG
- added X1, X2, X3, X4, X5, X6: PIN-1X-BIG, shrew-core:PAD-1X-BIG
- D1: value SK6812-EC20 -> 3V6; device shrew-core:SK6812-EC20 -> shrew-common:SOD-323
- L1: device shrew-common:C0402 -> shrew-common:0805
- moved U3 50.9 mm to (4.03, 5.50), turned to 270 degrees
- moved U4 39.3 mm to (13.4, 5.50), turned to 270 degrees
- moved ANT1 24.2 mm to (1.05, 15.5), flipped to the bottom, turned to 180 degrees
- moved D1 22.7 mm to (-2.60, 9.20)
- moved C4 9.80 mm to (2.40, 12.5), turned to 0 degrees
- moved ANT2 9.30 mm to (1.15, 19.9), turned to 180 degrees
- moved C3 8.58 mm to (2.40, 13.8), turned to 0 degrees
- moved FL1 8.32 mm to (1.40, 16.9), turned to 180 degrees
- moved C1 6.77 mm to (5.25, 13.1), turned to 90 degrees
- moved C7 6.63 mm to (9.00, 13.1), turned to 270 degrees
- moved C5 6.20 mm to (6.80, 21.9), turned to 180 degrees
- moved Y1 6.16 mm to (7.10, 13.1), turned to 180 degrees
- moved C2 5.99 mm to (9.00, 21.4), turned to 270 degrees
- moved L1 4.48 mm to (7.00, 20.5), turned to 180 degrees
- moved U2 3.22 mm to (5.00, 17.1), turned to 90 degrees
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Connections:
- new net +24V: C12.1, C13.1, C14.1, C15.1, C16.1, C18.1, C19.1, C20.1, IC1.3, R3.2, U3.5, U4.5, X5.1
- new net AUX1: JP1.3
- new net AUX2: JP1.2
- new net BATT-ADC: C17.1, D1.1, R2.2, R3.1
- new net N$10: C11.1, U4.8, X4.1
- new net N$13: JP2.3
- new net N$14: JP2.4
- new net N$4: C10.2, U3.6, X1.1
- new net N$5: C10.1, U3.8, X2.1
- new net N$8: C11.2, U4.6, X3.1
- net 3.3V: now also IC1.2, IC1.4, LED1.1, U3.4, U4.4; no longer D1.1
- net ESP-BOOT: now also JP2.2
- net GND: now also C12.2, C13.2, C14.2, C15.2, C16.2, C17.2, C18.2, C19.2, C20.2, D1.2, IC1.1, JP1.1, JP2.1, LED1.3, R2.1, U3.1, U3.7, U3.9, U4.1, U4.7, U4.9, U5.7, X6.1; no longer D1.3
- net RGBLED: now also LED1.4; no longer D1.4
Routing:
- net GND: track 22.8 -> 25.3 mm, vias 2 -> 8
- net N$8: track 0.00 -> 2.43 mm
- net N$10: track 0.00 -> 2.43 mm
- net N$5: track 0.00 -> 2.43 mm
- net N$4: track 0.00 -> 2.43 mm
- net N$1: track 0.00 -> 2.28 mm
- net N$7: track 0.00 -> 2.15 mm
- net 3.3V: track 5.85 -> 6.05 mm, vias 0 -> 2
- added copper zone on layer 1, net +24V
Other:
- board size 18 x 30 mm -> 18 x 25 mm
