File: electrical/shrew.sch (EAGLE design)
At the start: 20 parts, among them U1 ESP32-PICO-D4, U2 SX1280IMLTRT, U3 DRV8231DSGR, U4 DRV8231DSGR, Y1 OSCILLATOR-TG2016SMN

Commit message: wip, before splitting board into modules
Parts:
- added C10, C11: (no value), shrew-common:CAP0402-CAP
- added C12, C13, C14, C15, C16, C18, C19, C20: (no value), shrew-common:CAP0805
- added C17: 100n, shrew-common:CAP0402-CAP
- added FIDUCIAL1, FIDUCIAL2: FIDUCIAL-1MM-2MM, shrew-core:FIDUCIAL-1MM-2MM
- added IC1: (no value), shrew-common:V_REG_LM1117SOT223
- added JP1: (no value), shrew-common:M03PTH
- added JP2: (no value), shrew-common:M04PTH
- added JP3, JP4: (no value), shrew-common:M07-2MM-TH
- added LED1: SK6812-EC20, shrew-core:SK6812-EC20
- added R2: 10K, shrew-common:RESISTOR0402-RES
- added R3: 470K, shrew-common:RESISTOR0402-RES
- added TOOLING1, TOOLING2, TOOLING3: TOOLING-HOLE, shrew-core:TOOLING-HOLE
- added U5: DRV8244HQRYJRQ1, shrew-core:DRV8244SQRYJRQ1
- added X1, X2, X3, X4, X5, X6: PIN-1X-BIG, shrew-core:PIN-1X-BIG
- D1: value SK6812-EC20 -> 3V6; device shrew-core:SK6812-EC20 -> shrew-common:DIODE-ZENER-BZT52
- L1: device shrew-common:INDUCTOR0402 -> shrew-common:INDUCTOR0805
Connections:
- new net +24V: C12.1, C13.1, C14.1, C15.1, C16.1, C18.1, C19.1, C20.1, IC1.IN, R3.2, U3.VM, U4.VM, X5.P$1
- new net AUX1: JP1.3
- new net AUX2: JP1.2
- new net BATT-ADC: C17.1, D1.C, R2.2, R3.1
- new net N$10: C11.1, U4.OUT2, X4.P$1
- new net N$13: JP2.3
- new net N$14: JP2.4
- new net N$4: C10.2, U3.OUT1, X1.P$1
- new net N$5: C10.1, U3.OUT2, X2.P$1
- new net N$8: C11.2, U4.OUT1, X3.P$1
- net 3.3V: now also IC1.OUT, IC1.OUT@1, LED1.VDD, U3.VREF, U4.VREF; no longer D1.VDD
- net ESP-BOOT: now also JP2.2
- net GND: now also C12.2, C13.2, C14.2, C15.2, C16.2, C17.2, C18.2, C19.2, C20.2, D1.A, IC1.ADJ, JP1.1, JP2.1, LED1.VSS(GND), R2.1, U3.EPAD, U3.GND, U3.ISEN, U4.EPAD, U4.GND, U4.ISEN, U5.GND, X6.P$1; no longer D1.VSS(GND)
- net RGBLED: now also LED1.DIN; no longer D1.DIN
Other:
- note added: "10uF 50V typical"
- moved on the sheet: U3, U4
