File: electrical/shrew-rx.sch (EAGLE design)
At the start: 28 parts, among them U1 ESP32-PICO-D4, U2 SX1280IMLTRT, Y1 52MHz TCXO

Commit message: wip for rx
Parts:
- C12: value 470n -> DNP
- C17: value 100n -> 470n
Connections:
- net GND: now also U1.IO15/MTDO; no longer U1.IO15/MTDO(LOW)
- net OUT1: now also U1.SD3/IO10; no longer U1.SD3
- net OUT2: now also U1.SD2/IO9; no longer U1.SD2
- net U0RXD: now also U1.U0RXD(IO3); no longer U1.U0RXD
- net U0TXD: now also U1.U0TXD(IO1); no longer U1.U0TXD
Other:
- note added: "LOW = Quiet Boot"
- moved on the sheet: C13, R1
Changed lines of the file:
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@@
 <part name="P+15" library="shrew-common" deviceset="+24V" device=""/>
 <part name="GND22" library="shrew-common" deviceset="GND" device=""/>
-<part name="C17" library="shrew-common" deviceset="CAP" device="0402-CAP" value="100n"/>
+<part name="C17" library="shrew-common" deviceset="CAP" device="0402-CAP" value="470n"/>
 <part name="EDGE1" library="shrew-common" deviceset="M07" device="-2MM-TH"/>
 <part name="GND16" library="shrew-common" deviceset="GND" device=""/>
@@
 <part name="P+9" library="shrew-common" deviceset="3.3V" device=""/>
 <part name="GND20" library="shrew-common" deviceset="GND" device=""/>
-<part name="C12" library="shrew-common" deviceset="CAP" device="0402-CAP" value="470n"/>
+<part name="C12" library="shrew-common" deviceset="CAP" device="0402-CAP" value="DNP"/>
 </parts>
 <sheets>
@@
 <text x="17.78" y="10.16" size="1.27" layer="97">actually only for tweezers to squeeze</text>
 <text x="43.18" y="-10.16" size="1.27" layer="97" rot="R180">not actually +24V</text>
+<text x="43.18" y="43.18" size="1.27" layer="97" rot="R180">LOW = Quiet Boot</text>
+<text x="243.84" y="114.3" size="1.27" layer="97" rot="R180">not actually +24V</text>
 </plain>
 <instances>
@@
 <instance part="GND1" gate="1" x="45.72" y="38.1"/>
 <instance part="GND2" gate="1" x="114.3" y="20.32"/>
-<instance part="R1" gate="G$1" x="38.1" y="83.82" rot="R90"/>
-<instance part="P+2" gate="G$1" x="38.1" y="91.44"/>
+<instance part="R1" gate="G$1" x="48.26" y="83.82" rot="R90"/>
+<instance part="P+2" gate="G$1" x="48.26" y="91.44"/>
 <instance part="ANT1" gate="G$1" x="134.62" y="73.66"/>
 <instance part="FL1" gate="G$1" x="350.52" y="58.42"/>
@@
 <instance part="P+7" gate="G$1" x="259.08" y="109.22"/>
 <instance part="C10" gate="G$1" x="129.54" y="104.14"/>
-<instance part="C13" gate="G$1" x="27.94" y="71.12" rot="R180"/>
-<instance part="GND17" gate="1" x="27.94" y="60.96"/>
+<instance part="C13" gate="G$1" x="40.64" y="71.12" rot="R180"/>
+<instance part="GND17" gate="1" x="40.64" y="60.96"/>
 <instance part="EDGE2" gate="G$1" x="312.42" y="121.92" rot="R180"/>
 <instance part="P+8" gate="1" x="251.46" y="116.84"/>
@@
 </segment>
 <segment>
-<pinref part="U1" gate="G$1" pin="IO15/MTDO(LOW)"/>
+<pinref part="U1" gate="G$1" pin="IO15/MTDO"/>
 <wire x1="66.04" y1="43.18" x2="45.72" y2="43.18" width="0.1524" layer="91"/>
 <wire x1="45.72" y1="43.18" x2="45.72" y2="40.64" width="0.1524" layer="91"/>
@@
 <pinref part="GND17" gate="1" pin="GND"/>
 <pinref part="C13" gate="G$1" pin="1"/>
-<wire x1="27.94" y1="63.5" x2="27.94" y2="66.04" width="0.1524" layer="91"/>
+<wire x1="40.64" y1="63.5" x2="40.64" y2="66.04" width="0.1524" layer="91"/>
 </segment>
 <segment>
@@
 <pinref part="R1" gate="G$1" pin="2"/>
 <pinref part="P+2" gate="G$1" pin="3.3V"/>
-<wire x1="38.1" y1="88.9" x2="38.1" y2="91.44" width="0.1524" layer="91"/>
+<wire x1="48.26" y1="88.9" x2="48.26" y2="91.44" width="0.1524" layer="91"/>
 </segment>
 <segment>
@@
 <net name="U0TXD" class="0">
 <segment>
-<pinref part="U1" gate="G$1" pin="U0TXD"/>
+<pinref part="U1" gate="G$1" pin="U0TXD(IO1)"/>
 <wire x1="111.76" y1="91.44" x2="119.38" y2="91.44" width="0.1524" layer="91"/>
 <label x="119.38" y="91.44" size="1.27" layer="95" xref="yes"/>
@@
 <net name="U0RXD" class="0">
 <segment>
-<pinref part="U1" gate="G$1" pin="U0RXD"/>
+<pinref part="U1" gate="G$1" pin="U0RXD(IO3)"/>
 <wire x1="111.76" y1="88.9" x2="119.38" y2="88.9" width="0.1524" layer="91"/>
 <label x="119.38" y="88.9" size="1.27" layer="95" xref="yes"/>
@@
 <pinref part="U1" gate="G$1" pin="EN"/>
 <pinref part="R1" gate="G$1" pin="1"/>
-<wire x1="66.04" y1="76.2" x2="38.1" y2="76.2" width="0.1524" layer="91"/>
-<wire x1="38.1" y1="76.2" x2="38.1" y2="78.74" width="0.1524" layer="91"/>
-<wire x1="38.1" y1="76.2" x2="27.94" y2="76.2" width="0.1524" layer="91"/>
-<label x="20.32" y="76.2" size="1.27" layer="95" rot="R180" xref="yes"/>
+<wire x1="66.04" y1="76.2" x2="48.26" y2="76.2" width="0.1524" layer="91"/>
+<wire x1="48.26" y1="76.2" x2="48.26" y2="78.74" width="0.1524" layer="91"/>
+<wire x1="48.26" y1="76.2" x2="40.64" y2="76.2" width="0.1524" layer="91"/>
+<label x="30.48" y="76.2" size="1.27" layer="95" rot="R180" xref="yes"/>
 <pinref part="C13" gate="G$1" pin="2"/>
-<wire x1="27.94" y1="76.2" x2="20.32" y2="76.2" width="0.1524" layer="91"/>
-<wire x1="27.94" y1="73.66" x2="27.94" y2="76.2" width="0.1524" layer="91"/>
-<junction x="27.94" y="76.2"/>
-<junction x="38.1" y="76.2"/>
+<wire x1="40.64" y1="76.2" x2="30.48" y2="76.2" width="0.1524" layer="91"/>
+<wire x1="40.64" y1="73.66" x2="40.64" y2="76.2" width="0.1524" layer="91"/>
+<junction x="40.64" y="76.2"/>
+<junction x="48.26" y="76.2"/>
 </segment>
 </net>
@@
 </segment>
 <segment>
-<pinref part="U1" gate="G$1" pin="SD3"/>
+<pinref part="U1" gate="G$1" pin="SD3/IO10"/>
 <wire x1="111.76" y1="76.2" x2="116.84" y2="76.2" width="0.1524" layer="91"/>
 <label x="116.84" y="76.2" size="1.27" layer="95" xref="yes"/>
@@
 </segment>
 <segment>
-<pinref part="U1" gate="G$1" pin="SD2"/>
+<pinref part="U1" gate="G$1" pin="SD2/IO9"/>
 <wire x1="111.76" y1="78.74" x2="116.84" y2="78.74" width="0.1524" layer="91"/>
 <label x="116.84" y="78.74" size="1.27" layer="95" xref="yes"/>

Commit message: schematic stitcher
Connections:
- net +24V renamed V-ADC
- net OUT1 renamed SIG4
- net OUT2 renamed SIG3
- net OUT3 renamed SIG2
- net OUT4 renamed SIG1
Changed lines of the file:
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@@
-</segment>
-</net>
-<net name="+24V" class="0">
-<segment>
-<pinref part="P+15" gate="1" pin="+24V"/>
-<pinref part="R3" gate="G$1" pin="2"/>
-<wire x1="48.26" y1="-7.62" x2="48.26" y2="-10.16" width="0.1524" layer="91"/>
-</segment>
-<segment>
-<pinref part="EDGE1" gate="G$1" pin="5"/>
-<wire x1="276.86" y1="116.84" x2="256.54" y2="116.84" width="0.1524" layer="91"/>
-<wire x1="256.54" y1="116.84" x2="256.54" y2="111.76" width="0.1524" layer="91"/>
-<pinref part="P+8" gate="1" pin="+24V"/>
-<wire x1="256.54" y1="111.76" x2="251.46" y2="111.76" width="0.1524" layer="91"/>
-<wire x1="251.46" y1="111.76" x2="251.46" y2="114.3" width="0.1524" layer="91"/>
 </segment>
 </net>
@@
 </segment>
 </net>
-<net name="OUT1" class="0">
-<segment>
-<pinref part="EDGE1" gate="G$1" pin="1"/>
-<wire x1="276.86" y1="127" x2="269.24" y2="127" width="0.1524" layer="91"/>
-<label x="269.24" y="127" size="1.27" layer="95" rot="R180" xref="yes"/>
-</segment>
-<segment>
-<pinref part="U1" gate="G$1" pin="SD3/IO10"/>
-<wire x1="111.76" y1="76.2" x2="116.84" y2="76.2" width="0.1524" layer="91"/>
-<label x="116.84" y="76.2" size="1.27" layer="95" xref="yes"/>
-</segment>
-</net>
-<net name="OUT2" class="0">
+<net name="SIG3" class="0">
 <segment>
 <pinref part="EDGE1" gate="G$1" pin="2"/>
@@
 </segment>
 </net>
-<net name="OUT3" class="0">
+<net name="SIG2" class="0">
 <segment>
 <pinref part="EDGE1" gate="G$1" pin="3"/>
@@
 </segment>
 </net>
-<net name="OUT4" class="0">
+<net name="SIG1" class="0">
 <segment>
 <pinref part="EDGE1" gate="G$1" pin="4"/>
@@
 </segment>
 </net>
+<net name="SIG4" class="0">
+<segment>
+<pinref part="U1" gate="G$1" pin="SD3/IO10"/>
+<wire x1="111.76" y1="76.2" x2="116.84" y2="76.2" width="0.1524" layer="91"/>
+<label x="116.84" y="76.2" size="1.27" layer="95" xref="yes"/>
+</segment>
+<segment>
+<pinref part="EDGE1" gate="G$1" pin="1"/>
+<wire x1="276.86" y1="127" x2="269.24" y2="127" width="0.1524" layer="91"/>
+<label x="269.24" y="127" size="1.27" layer="95" rot="R180" xref="yes"/>
+</segment>
+</net>
+<net name="V-ADC" class="0">
+<segment>
+<pinref part="EDGE1" gate="G$1" pin="5"/>
+<wire x1="276.86" y1="116.84" x2="256.54" y2="116.84" width="0.1524" layer="91"/>
+<wire x1="256.54" y1="116.84" x2="256.54" y2="111.76" width="0.1524" layer="91"/>
+<pinref part="P+8" gate="1" pin="+24V"/>
+<wire x1="256.54" y1="111.76" x2="251.46" y2="111.76" width="0.1524" layer="91"/>
+<wire x1="251.46" y1="111.76" x2="251.46" y2="114.3" width="0.1524" layer="91"/>
+</segment>
+<segment>
+<pinref part="P+15" gate="1" pin="+24V"/>
+<pinref part="R3" gate="G$1" pin="2"/>
+<wire x1="48.26" y1="-7.62" x2="48.26" y2="-10.16" width="0.1524" layer="91"/>
+</segment>
+</net>

Commit message: changed all 0402 footprints on rx
Parts:
- C1, C10, C13, C17, C2, C3, C4, C5, C6, C7, C8, C9: device shrew-common:CAP0402-CAP -> shrew-common:CAP0402-REV
- R1, R2, R3: device shrew-common:RESISTOR0402-RES -> shrew-common:RESISTOR0402-REV
