File: electrical/shrew-mega-integrated.brd (EAGLE design)
At the start: 18 x 27 mm, 48 parts, among them U1 ESP32-PICO-D4, U2 SX1280IMLTRT, U3 DRV8244SQRYJRQ1, U4 DRV8244SQRYJRQ1, X1 PIN-1X-BIG, X2 PIN-1X-BIG, X3 PIN-1X-BIG, X4 PIN-1X-BIG, X5 PIN-1X-BIG, X6 PIN-1X-BIG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

Commit message: wip
Parts:
- added C26: 100n, shrew-common:0402-REV
- added C27: 10u, shrew-common:0805
- added D2: (no value), shrew-common:SOD-323
- added L2: 6u8, shrew-common:0805
- C24, C25: value (none) -> 10u
- IC1: value (none) -> LMR16006YQ3DDCTQ1; device shrew-common:SOT223 -> shrew-core:SOT95P280X110-6N
- moved C24 9.50 mm to (9.00, 9.90), flipped to the top, turned to 90 degrees
- moved C21 5.52 mm to (16.4, 7.15)
- moved C25 4.09 mm to (12.9, 11.1), flipped to the bottom
- moved C22 1.60 mm to (16.4, 5.55)
- moved C23 1.60 mm to (16.4, 3.95)
- moved IC1 1.39 mm to (8.50, 6.60), turned to 90 degrees
- renumbered EDGE2 to EDGE1
Connections:
- new net N$10: C26.1, D2.1, IC1.6, L2.1
- new net N$4: C26.2, IC1.1
- net +24V: now also C21.1, IC1.4, IC1.5; no longer C25.1, IC1.1
- net 3.3V: now also C25.1, C27.1, L2.2; no longer C21.1
- net GND: now also C27.2, D2.2; no longer IC1.4
Routing:
- net 3.3V: track 38.1 -> 51.1 mm
- net N$10: track 0.00 -> 3.83 mm
- net GND: track 45.3 -> 42.2 mm, vias 58 -> 59
- net N$4: track 0.00 -> 1.97 mm
- net RADIO-RST: track 33.2 -> 31.9 mm
- net +24V: track 24.9 -> 26.1 mm
- net SIG1: track 17.7 -> 18.3 mm
Other:
- board text removed: "G"
