File: electrical/shrew-mega-integrated.sch (EAGLE design)
At the start: 28 parts, among them U1 ESP32-PICO-D4, U2 SX1280IMLTRT, Y1 52MHz TCXO

Commit message: initial work on integrated versions
Parts:
- removed EDGE1: (no value), shrew-common:M07-2MM-TH
- added C14, C15: (no value), shrew-common:CAP0402-CAP
- added C16, C18, C19, C20, C21, C22, C23, C24, C25: (no value), shrew-common:CAP0805
- added IC1: (no value), shrew-common:V_REG_SOT-SOT223
- added R4: (no value), shrew-common:RESISTOR0402-RES
- added U3, U4: DRV8244SQRYJRQ1, shrew-core:DRV8244SQRYJRQ1
- added X1, X2, X3, X4, X5, X6: PIN-1X-BIG, shrew-core:PIN-1X-BIG
Connections:
- new net +24V: C16.1, C18.1, C19.1, C20.1, C22.1, C23.1, C24.1, C25.1, IC1.IN, R4.2, U3.VM, U4.VM, X5.P$1
- new net MOTOR1: C14.1, U3.OUT1, U3.OUT1_2, X2.P$1
- new net MOTOR2: C14.2, U3.OUT2, U3.OUT2_2, X1.P$1
- new net MOTOR3: C15.1, U4.OUT1, U4.OUT1_2, X4.P$1
- new net MOTOR4: C15.2, U4.OUT2, U4.OUT2_2, X3.P$1
- net 3.3V: now also C21.1, IC1.VO; no longer EDGE1.6
- net GND: now also C16.2, C18.2, C19.2, C20.2, C21.2, C22.2, C23.2, C24.2, C25.2, IC1.GND, IC1.TAB, U3.DIAG, U3.DRVOFF, U3.GND, U3.IPROPI, U3.ITRIP, U3.SR, U4.DIAG, U4.DRVOFF, U4.GND, U4.IPROPI, U4.ITRIP, U4.SR, X6.P$1; no longer EDGE1.7
- net RADIO-RST: now also U3.SLEEP_N, U4.SLEEP_N
- net SIG1: now also U4.EN_IN1; no longer EDGE1.4
- net SIG2: now also U4.PH_IN2; no longer EDGE1.3
- net SIG3: now also U3.EN_IN1; no longer EDGE1.2
- net SIG4: now also U3.PH_IN2; no longer EDGE1.1
- net V-ADC: now also R4.1; no longer EDGE1.5
Other:
- note added: "10uF 50V typical"
- note added: "Current regulation disabled, OCP still used"
- note added: "Default slew rate 22V/us"
- note added: "Faults cause retry automatically"
- note added: "PWM mode"
- moved on the sheet: C17, D1, R2, R3

Commit message: wip
Parts:
- removed EDGE2: (no value), shrew-common:M05PTH
- added C26: 100n, shrew-common:CAP0402-REV
- added C27: 10u, shrew-common:CAP0805
- added D2: (no value), shrew-common:DIODESOD
- added EDGE1: (no value), shrew-common:M05PTH
- added L2: 6u8, shrew-common:INDUCTOR0805
- C24, C25: value (none) -> 10u
- IC1: value (none) -> LMR16006YQ3DDCTQ1; device shrew-common:V_REG_SOT-SOT223 -> shrew-core:LMR16006XDDCR
Connections:
- new net N$10: C26.1, D2.C, IC1.SW, L2.1
- new net N$4: C26.2, IC1.CB
- net +24V: now also C21.1, IC1.SHDN, IC1.VIN; no longer C25.1, IC1.IN
- net 3.3V: now also C25.1, C27.1, IC1.FB, L2.2; no longer C21.1, IC1.VO
- net AUX1: now also EDGE1.1; no longer EDGE2.1
- net AUX2: now also EDGE1.2; no longer EDGE2.2
- net GND: now also C27.2, D2.A, EDGE1.5; no longer EDGE2.5, IC1.TAB
- net U0RXD: now also EDGE1.3; no longer EDGE2.3
- net U0TXD: now also EDGE1.4; no longer EDGE2.4
Other:
- moved on the sheet: C21, C22, C23, C24, C25
