File: electrical/shrew-mini.sch (EAGLE design)
At the start: 18 parts, among them IC1 Vreg +3V3, U1 DRV8231DSGR, U2 DRV8231DSGR, X1 PIN-1X-BIG, X2 PIN-1X-BIG, X3 PIN-1X-BIG, X4 PIN-1X-BIG, X5 PIN-1X-1.5MMSQ, X6 PIN-1X-1.5MMSQ

Commit message: schematic stitcher
Connections:
- net N$10 renamed MOTOR2
- net N$4 renamed MOTOR3
- net N$5 renamed MOTOR4
- net N$7 renamed V-ADC
- net N$8 renamed MOTOR1
Changed lines of the file:
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@@
 <wire x1="45.72" y1="17.78" x2="48.26" y2="17.78" width="0.1524" layer="91"/>
 <wire x1="48.26" y1="17.78" x2="48.26" y2="15.24" width="0.1524" layer="91"/>
+<junction x="48.26" y="15.24"/>
+<junction x="48.26" y="12.7"/>
 </segment>
 <segment>
@@
 <wire x1="45.72" y1="53.34" x2="48.26" y2="53.34" width="0.1524" layer="91"/>
 <wire x1="48.26" y1="53.34" x2="48.26" y2="50.8" width="0.1524" layer="91"/>
+<junction x="48.26" y="50.8"/>
+<junction x="48.26" y="48.26"/>
 </segment>
 <segment>
@@
 </segment>
 </net>
-<net name="N$4" class="0">
+<net name="MOTOR3" class="0">
 <segment>
 <pinref part="U2" gate="A" pin="OUT1"/>
@@
 </segment>
 </net>
-<net name="N$5" class="0">
+<net name="MOTOR4" class="0">
 <segment>
 <pinref part="U2" gate="A" pin="OUT2"/>
@@
 </segment>
 </net>
-<net name="N$8" class="0">
+<net name="MOTOR1" class="0">
 <segment>
 <pinref part="U1" gate="A" pin="OUT1"/>
@@
 </segment>
 </net>
-<net name="N$10" class="0">
+<net name="MOTOR2" class="0">
 <segment>
 <pinref part="U1" gate="A" pin="OUT2"/>
@@
 </segment>
 </net>
-<net name="N$7" class="0">
+<net name="V-ADC" class="0">
 <segment>
 <pinref part="JP1" gate="G$1" pin="3"/>

Commit message: added power input silk
Parts:
- X6: value PIN-1X-1.5MMSQ -> PIN-1X-MED; device shrew-core:PIN-1X-1.5MMSQ -> shrew-core:PIN-1X-MED
Changed lines of the file:
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@@
 <grid distance="0.1" unitdist="inch" unit="inch" style="lines" multiple="1" display="no" altdistance="0.01" altunitdist="inch" altunit="inch"/>
 <layers>
-<layer number="1" name="Top" color="4" fill="1" visible="no" active="no"/>
-<layer number="2" name="Route2" color="1" fill="3" visible="no" active="no"/>
-<layer number="3" name="Route3" color="4" fill="3" visible="no" active="no"/>
-<layer number="4" name="Route4" color="1" fill="4" visible="no" active="no"/>
-<layer number="5" name="Route5" color="4" fill="4" visible="no" active="no"/>
-<layer number="6" name="Route6" color="1" fill="8" visible="no" active="no"/>
-<layer number="7" name="Route7" color="4" fill="8" visible="no" active="no"/>
-<layer number="8" name="Route8" color="1" fill="2" visible="no" active="no"/>
-<layer number="9" name="Route9" color="4" fill="2" visible="no" active="no"/>
-<layer number="10" name="Route10" color="1" fill="7" visible="no" active="no"/>
-<layer number="11" name="Route11" color="4" fill="7" visible="no" active="no"/>
-<layer number="12" name="Route12" color="1" fill="5" visible="no" active="no"/>
-<layer number="13" name="Route13" color="4" fill="5" visible="no" active="no"/>
-<layer number="14" name="Route14" color="1" fill="6" visible="no" active="no"/>
-<layer number="15" name="Route15" color="4" fill="6" visible="no" active="no"/>
-<layer number="16" name="Bottom" color="1" fill="1" visible="no" active="no"/>
-<layer number="17" name="Pads" color="2" fill="1" visible="no" active="no"/>
-<layer number="18" name="Vias" color="2" fill="1" visible="no" active="no"/>
-<layer number="19" name="Unrouted" color="6" fill="1" visible="no" active="no"/>
-<layer number="20" name="Dimension" color="15" fill="1" visible="no" active="no"/>
-<layer number="21" name="tPlace" color="7" fill="1" visible="no" active="no"/>
-<layer number="22" name="bPlace" color="7" fill="1" visible="no" active="no"/>
-<layer number="23" name="tOrigins" color="15" fill="1" visible="no" active="no"/>
-<layer number="24" name="bOrigins" color="15" fill="1" visible="no" active="no"/>
-<layer number="25" name="tNames" color="7" fill="1" visible="no" active="no"/>
-<layer number="26" name="bNames" color="7" fill="1" visible="no" active="no"/>
-<layer number="27" name="tValues" color="7" fill="1" visible="no" active="no"/>
-<layer number="28" name="bValues" color="7" fill="1" visible="no" active="no"/>
+<layer number="1" name="Top" color="4" fill="1" visible="yes" active="no"/>
+<layer number="2" name="Route2" color="1" fill="3" visible="yes" active="no"/>
+<layer number="3" name="Route3" color="4" fill="3" visible="yes" active="no"/>
+<layer number="4" name="Route4" color="1" fill="4" visible="yes" active="no"/>
+<layer number="5" name="Route5" color="4" fill="4" visible="yes" active="no"/>
+<layer number="6" name="Route6" color="1" fill="8" visible="yes" active="no"/>
+<layer number="7" name="Route7" color="4" fill="8" visible="yes" active="no"/>
+<layer number="8" name="Route8" color="1" fill="2" visible="yes" active="no"/>
+<layer number="9" name="Route9" color="4" fill="2" visible="yes" active="no"/>
+<layer number="10" name="Route10" color="1" fill="7" visible="yes" active="no"/>
+<layer number="11" name="Route11" color="4" fill="7" visible="yes" active="no"/>
+<layer number="12" name="Route12" color="1" fill="5" visible="yes" active="no"/>
+<layer number="13" name="Route13" color="4" fill="5" visible="yes" active="no"/>
+<layer number="14" name="Route14" color="1" fill="6" visible="yes" active="no"/>
+<layer number="15" name="Route15" color="4" fill="6" visible="yes" active="no"/>
+<layer number="16" name="Bottom" color="1" fill="1" visible="yes" active="no"/>
+<layer number="17" name="Pads" color="2" fill="1" visible="yes" active="no"/>
+<layer number="18" name="Vias" color="2" fill="1" visible="yes" active="no"/>
+<layer number="19" name="Unrouted" color="6" fill="1" visible="yes" active="no"/>
+<layer number="20" name="Dimension" color="15" fill="1" visible="yes" active="no"/>
+<layer number="21" name="tPlace" color="7" fill="1" visible="yes" active="no"/>
+<layer number="22" name="bPlace" color="7" fill="1" visible="yes" active="no"/>
+<layer number="23" name="tOrigins" color="15" fill="1" visible="yes" active="no"/>
+<layer number="24" name="bOrigins" color="15" fill="1" visible="yes" active="no"/>
+<layer number="25" name="tNames" color="7" fill="1" visible="yes" active="no"/>
+<layer number="26" name="bNames" color="7" fill="1" visible="yes" active="no"/>
+<layer number="27" name="tValues" color="7" fill="1" visible="yes" active="no"/>
+<layer number="28" name="bValues" color="7" fill="1" visible="yes" active="no"/>
 <layer number="29" name="tStop" color="7" fill="3" visible="no" active="no"/>
 <layer number="30" name="bStop" color="7" fill="6" visible="no" active="no"/>
@@
 <layer number="35" name="tGlue" color="7" fill="4" visible="no" active="no"/>
 <layer number="36" name="bGlue" color="7" fill="5" visible="no" active="no"/>
-<layer number="37" name="tTest" color="7" fill="1" visible="no" active="no"/>
-<layer number="38" name="bTest" color="7" fill="1" visible="no" active="no"/>
+<layer number="37" name="tTest" color="7" fill="1" visible="yes" active="no"/>
+<layer number="38" name="bTest" color="7" fill="1" visible="yes" active="no"/>
 <layer number="39" name="tKeepout" color="4" fill="11" visible="no" active="no"/>
 <layer number="40" name="bKeepout" color="1" fill="11" visible="no" active="no"/>
@@
 <layer number="44" name="Drills" color="7" fill="1" visible="no" active="no"/>
 <layer number="45" name="Holes" color="7" fill="1" visible="no" active="no"/>
-<layer number="46" name="Milling" color="3" fill="1" visible="no" active="no"/>
-<layer number="47" name="Measures" color="7" fill="1" visible="no" active="no"/>
-<layer number="48" name="Document" color="7" fill="1" visible="no" active="no"/>
-<layer number="49" name="Reference" color="7" fill="1" visible="no" active="no"/>
-<layer number="50" name="dxf" color="7" fill="1" visible="no" active="no"/>
-<layer number="51" name="tDocu" color="7" fill="1" visible="no" active="no"/>
-<layer number="52" name="bDocu" color="7" fill="1" visible="no" active="no"/>
-<layer number="53" name="tGND_GNDA" color="7" fill="9" visible="no" active="no"/>
-<layer number="54" name="bGND_GNDA" color="1" fill="9" visible="no" active="no"/>
-<layer number="56" name="wert" color="7" fill="1" visible="no" active="no"/>
+<layer number="46" name="Milling" color="3" fill="1" visible="yes" active="no"/>
+<layer number="47" name="Measures" color="7" fill="1" visible="yes" active="no"/>
+<layer number="48" name="Document" color="7" fill="1" visible="yes" active="no"/>
+<layer number="49" name="Reference" color="7" fill="1" visible="yes" active="no"/>
+<layer number="50" name="dxf" color="7" fill="1" visible="yes" active="no"/>
+<layer number="51" name="tDocu" color="7" fill="1" visible="yes" active="no"/>
+<layer number="52" name="bDocu" color="7" fill="1" visible="yes" active="no"/>
+<layer number="53" name="tGND_GNDA" color="7" fill="9" visible="yes" active="no"/>
+<layer number="54" name="bGND_GNDA" color="1" fill="9" visible="yes" active="no"/>
+<layer number="56" name="wert" color="7" fill="1" visible="yes" active="no"/>
 <layer number="90" name="Modules" color="5" fill="1" visible="yes" active="yes"/>
 <layer number="91" name="Nets" color="2" fill="1" visible="yes" active="yes"/>
@@
 <layer number="97" name="Info" color="7" fill="1" visible="yes" active="yes"/>
 <layer number="98" name="Guide" color="6" fill="1" visible="yes" active="yes"/>
+<layer number="99" name="SpiceOrder" color="5" fill="1" visible="no" active="no"/>
 <layer number="100" name="Muster" color="7" fill="1" visible="no" active="no"/>
 <layer number="101" name="Patch_Top" color="12" fill="4" visible="no" active="yes"/>
@@
 <part name="P+13" library="shrew-common" deviceset="3.3V" device=""/>
 <part name="GND18" library="shrew-common" deviceset="GND" device=""/>
-<part name="X6" library="shrew-core" deviceset="PIN-1X" device="-1.5MMSQ" value="PIN-1X-1.5MMSQ"/>
+<part name="X6" library="shrew-core" deviceset="PIN-1X" device="-MED" value="PIN-1X-MED"/>
 <part name="GND19" library="shrew-common" deviceset="GND" device=""/>
 <part name="C1" library="shrew-common" deviceset="CAP" device="0805"/>

Commit message: up-rev
Parts:
- added ANT1, ANT2: 74889302450, shrew-common:ANTENNA2SMD
- added C10, C8, C9: 100n, shrew-common:CAP0402-REV
- added C11: 10uF 25V, shrew-common:CAP0805
- added C12: DNP, shrew-common:CAP0402-CAP
- added C13, C17: 470n, shrew-common:CAP0402-REV
- added C14, C15: (no value), shrew-common:CAP0402-CAP
- added C16, C18, C19, C20, C21: (no value), shrew-common:CAP0805
- added D1: 3V6, shrew-common:DIODE-ZENER-BZT52
- added EDGE1: (no value), shrew-common:M05PTH
- added FL1: 2450FM07D0034T, shrew-core:2450FM07D0034T
- added L1: 15u, shrew-common:INDUCTOR0805
- added LED1: SK6812-EC20, shrew-core:SK6812-EC20
- added R2, R3: 10K, shrew-common:RESISTOR0402-REV
- added R4: (no value), shrew-common:RESISTOR0402-RES
- added U3, U4: DRV8231DSGR, shrew-core:DRV8231DSGR
- added X7, X8: PIN-1X-MED, shrew-core:PIN-1X-MED
- added Y1: 52MHz TCXO, shrew-common:OSCILLATOR-TG2016SMN
- C1: value (none) -> 1n; device shrew-common:CAP0805 -> shrew-common:CAP0402-REV
- C2: value (none) -> 470n; device shrew-common:CAP0805 -> shrew-common:CAP0402-REV
- C3, C4: value (none) -> 10n; device shrew-common:CAP0805 -> shrew-common:CAP0402-REV
- C5: value (none) -> 100n; device shrew-common:CAP0805 -> shrew-common:CAP0402-REV
- C6, C7: value (none) -> 100n; device shrew-common:CAP0402-CAP -> shrew-common:CAP0402-REV
- JP1: device shrew-common:M07-2MM-TH -> shrew-common:M07-2MM-TH-TINY
- R1: value (none) -> 10K; device shrew-common:RESISTOR0402-RES -> shrew-common:RESISTOR0402-REV
- U1: value DRV8231DSGR -> ESP32-PICO-D4; device shrew-core:DRV8231DSGR -> shrew-core:ESP32-PICO-D4
- U2: value DRV8231DSGR -> SX1280IMLTRT; device shrew-core:DRV8231DSGR -> shrew-core:SX1280IMLTRT
- X5: value PIN-1X-1.5MMSQ -> PIN-1X-MED; device shrew-core:PIN-1X-1.5MMSQ -> shrew-core:PIN-1X-MED
Connections:
- new net AUX1: EDGE1.1, U1.IO19
- new net AUX2: EDGE1.2, U1.IO22
- new net BATT-ADC: C17.1, D1.C, R2.2, R3.1, U1.IO4
- new net ESP-BOOT: C12.2, U1.IO0(BOOT)
- new net ESP-EN: C13.2, R1.1, U1.EN
- new net N$1: ANT1.SIGNAL, U1.LNA_IN
- new net N$11: C3.2, U2.VR_PA
- new net N$2: C1.1, Y1.OUT
- new net N$3: C1.2, U2.XTA
- new net N$5: U1.IO14
- new net N$6: FL1.IN, U2.RFIO
- new net N$7: ANT2.SIGNAL, FL1.OUT
- new net N$8: U1.IO2
- new net N$9: L1.2, U2.DCC_SW
- new net RADIO-BUSY: U1.IO23, U2.BUSY
- new net RADIO-CS: U1.IO32, U2.NSS_CTS
- new net RADIO-DIO: U1.IO18, U2.DIO1
- new net RADIO-RST: U1.IO21, U2.NRESET
- new net RADIO-VDD: C2.2, C4.2, L1.1, U2.DCC_FB, U2.VDD_INN
- new net RGBLED: LED1.DIN, U1.IO5
- new net SPI-MISO: U1.IO26, U2.MISO_TX
- new net SPI-MOSI: U1.IO25, U2.MOSI_RX
- new net SPI-SCK: U1.IO33, U2.SCK_RTSN
- new net U0RXD: EDGE1.3, U1.U0RXD(IO3)
- new net U0TXD: EDGE1.4, U1.U0TXD(IO1)
- net +24V: now also C16.1, C18.1, C19.1, C20.1, R4.2, U3.VM, U4.VM, X7.P$1; no longer C1.1, C2.1, C3.1, C4.1, R1.2, U1.VM, U2.VM
- net 3.3V: now also C10.1, C11.1, C21.1, C5.2, C6.2, C7.2, C8.1, C9.1, LED1.VDD, R1.2, U1.VDD3P3_CPU, U1.VDD3P3_RTC, U1.VDDA, U1.VDDA3P3, U1.VDD_SDIO, U2.VBAT, U2.VBAT_IO, U3.VREF, U4.VREF, Y1.VCC; no longer C5.1, U1.VREF, U2.VREF
- net GND: now also C10.2, C11.2, C12.1, C13.1, C16.2, C17.2, C18.2, C19.2, C2.1, C20.2, C21.2, C3.1, C4.1, C5.1, C6.1, C7.1, C8.2, C9.2, D1.A, EDGE1.5, LED1.VSS(GND), R2.1, U1.IO15/MTDO, U2.GND_2, U2.GND_3, U2.GND_4, U2.GND_5, U2.GND_6, U2.GND_7, U3.EPAD, U3.GND, U3.ISEN, U4.EPAD, U4.GND, U4.ISEN, X8.P$1, Y1.GND; no longer C1.2, C2.2, C3.2, C4.2, C5.2, U1.EPAD, U1.ISEN, U2.EPAD, U2.ISEN
- net MOTOR1: now also C15.2, U4.OUT1; no longer C7.2, U1.OUT1
- net MOTOR2: now also C15.1, U4.OUT2; no longer C7.1, U1.OUT2
- net MOTOR3: now also C14.2, U3.OUT1; no longer C6.2, U2.OUT1
- net MOTOR4: now also C14.1, U3.OUT2; no longer C6.1, U2.OUT2
- net SIG1: now also U1.IO13, U4.IN2; no longer U1.IN2
- net SIG2: now also U1.IO27, U4.IN1; no longer U1.IN1
- net SIG3: now also U1.SD2/IO9, U3.IN2; no longer U2.IN2
- net SIG4: now also U1.SD3/IO10, U3.IN1; no longer U2.IN1
- net V-ADC: now also R3.2, R4.1; no longer R1.1
Other:
- note added: "LOW = Quiet Boot"
- note added: "actually only for tweezers to squeeze"
- note added: "not actually +24V"
- moved on the sheet: C1, C2, C3, C4, C5, C6, C7, IC1, JP1, R1
