File: electrical/shrew-mega.brd (EAGLE design)
At the start: 18 x 15 mm, 22 parts, among them U1 DRV8244SQRYJRQ1, U2 DRV8244SQRYJRQ1, X1 PIN-1X-BIG, X2 PIN-1X-BIG, X3 PIN-1X-BIG, X4 PIN-1X-BIG, X5 PIN-1X-BIG, X6 PIN-1X-BIG

Commit message: up-rev
Parts:
- removed JP1: (no value), shrew-common:1X07-2MM-TH
- added ANT1, ANT2: 74889302450, shrew-common:ANTENNA-CHIP2
- added C12: DNP, shrew-common:0402-CAP
- added C13, C17: 470n, shrew-common:0402-REV
- added C14, C15: (no value), shrew-common:0402-CAP
- added C16, C18, C19, C20, C21, C22, C23: (no value), shrew-common:0805
- added C24, C25, C27: 10u, shrew-common:0805
- added C26: 100n, shrew-common:0402-REV
- added D1: 3V6, shrew-common:SOD-323
- added D2: (no value), shrew-common:SOD-323
- added EDGE1: (no value), shrew-common:1X05
- added FL1: 2450FM07D0034T, shrew-core:FIL_2450FM07D0034T
- added L1: 15u, shrew-common:0805
- added L2: 6u8, shrew-common:0805
- added LED1: SK6812-EC20, shrew-core:SK6812-EC20
- added R2, R3: 10K, shrew-common:0402-REV
- added R4: (no value), shrew-common:0402-RES
- added U3, U4: DRV8244SQRYJRQ1, shrew-core:RYJ0016A-MFG
- added Y1: 52MHz TCXO, shrew-common:OSC_TG2016SMN_50.0000M-ECGNNMB
- C1: value (none) -> 1n; device shrew-common:0805 -> shrew-common:0402-REV
- C10, C9: value (none) -> 100n; device shrew-common:0402-CAP -> shrew-common:0402-REV
- C11: value (none) -> 10uF 25V
- C2: value (none) -> 470n; device shrew-common:0805 -> shrew-common:0402-REV
- C3, C4: value (none) -> 10n; device shrew-common:0805 -> shrew-common:0402-REV
- C5, C6, C7, C8: value (none) -> 100n; device shrew-common:0805 -> shrew-common:0402-REV
- IC1: value (none) -> LMR16006YQ3DDCTQ1; device shrew-common:SOT223 -> shrew-core:SOT95P280X110-6N
- R1: value (none) -> 10K; device shrew-common:0402-RES -> shrew-common:0402-REV
- U1: value DRV8244SQRYJRQ1 -> ESP32-PICO-D4; device shrew-core:RYJ0016A-MFG -> shrew-core:PQFN50P700X700X104-49N
- U2: value DRV8244SQRYJRQ1 -> SX1280IMLTRT; device shrew-core:RYJ0016A-MFG -> shrew-core:QFN24_4X4_SEM
- moved C10 22.7 mm to (6.50, 24.7), flipped to the bottom, turned to 90 degrees
- moved C9 19.8 mm to (14.3, 20.2), flipped to the bottom, turned to 90 degrees
- moved C1 18.1 mm to (6.60, 21.8), flipped to the top, turned to 0 degrees
- moved C3 18.0 mm to (7.30, 24.6), flipped to the top, turned to 270 degrees
- moved C2 17.6 mm to (14.8, 17.7), flipped to the top
- moved C7 17.1 mm to (6.60, 18.0), flipped to the top
- moved C4 16.0 mm to (6.00, 24.6), flipped to the top
- moved R1 15.7 mm to (12.6, 24.7), turned to 180 degrees
- moved U2 14.7 mm to (10.6, 22.0)
- moved C6 13.8 mm to (11.8, 18.6), flipped to the top
- moved U1 13.4 mm to (10.1, 20.0), flipped to the bottom, turned to 270 degrees
- moved C5 13.1 mm to (15.9, 20.2), flipped to the top, turned to 90 degrees
- moved C8 13.0 mm to (9.20, 24.2)
- moved C11 6.20 mm to (10.1, 16.0), turned to 180 degrees
- moved IC1 1.39 mm to (8.50, 6.60), turned to 90 degrees
Connections:
- removed net SLEEP: U1.3, U2.3
- new net AUX1: EDGE1.1, U1.38
- new net AUX2: EDGE1.2, U1.39
- new net BATT-ADC: C17.1, D1.1, R2.2, R3.1, U1.24
- new net ESP-BOOT: C12.2, U1.23
- new net ESP-EN: C13.2, R1.1, U1.9
- new net N$1: ANT1.FEED, U1.2
- new net N$10: C26.1, D2.1, IC1.6, L2.1
- new net N$11: C3.2, U2.1
- new net N$2: C1.1, Y1.3
- new net N$3: C1.2, U2.4
- new net N$4: C26.2, IC1.1
- new net N$5: U1.17
- new net N$6: FL1.1, U2.22
- new net N$7: ANT2.FEED, FL1.3
- new net N$8: U1.22
- new net N$9: L1.2, U2.14
- new net RADIO-BUSY: U1.36, U2.7
- new net RADIO-CS: U1.12, U2.19
- new net RADIO-DIO: U1.35, U2.8
- new net RADIO-RST: U1.42, U2.3, U3.3, U4.3
- new net RADIO-VDD: C2.2, C4.2, L1.1, U2.12, U2.2
- new net RGBLED: LED1.4, U1.34
- new net SPI-MISO: U1.15, U2.16
- new net SPI-MOSI: U1.14, U2.17
- new net SPI-SCK: U1.13, U2.18
- new net U0RXD: EDGE1.3, U1.40
- new net U0TXD: EDGE1.4, U1.41
- net +24V: now also C16.1, C18.1, C19.1, C20.1, C21.1, C22.1, C23.1, C24.1, IC1.4, IC1.5, R4.2, U3.4, U4.4; no longer C1.1, C11.1, C2.1, C3.1, C4.1, C5.1, C6.1, C7.1, IC1.1, R1.2, U1.4, U2.4
- net 3.3V: now also C10.1, C11.1, C25.1, C27.1, C5.2, C6.2, C7.2, C9.1, L2.2, LED1.1, R1.2, U1.1, U1.19, U1.26, U1.3, U1.37, U1.4, U1.43, U1.46, U2.11, U2.15, Y1.4; no longer JP1.2
- net GND: now also C10.2, C12.1, C13.1, C16.2, C17.2, C18.2, C19.2, C2.1, C20.2, C21.2, C22.2, C23.2, C24.2, C25.2, C27.2, C3.1, C4.1, C5.1, C6.1, C7.1, C9.2, D1.2, D2.2, EDGE1.5, FL1.2, FL1.4, LED1.3, R2.1, U1.21, U1.49, U2.20, U2.21, U2.23, U2.24, U2.25, U2.5, U3.10, U3.13, U3.14, U3.15, U3.2, U3.7, U4.10, U4.13, U4.14, U4.15, U4.2, U4.7, Y1.2; no longer C1.2, C2.2, C3.2, C4.2, C5.2, C6.2, C7.2, IC1.4, JP1.1, U1.10, U1.13, U1.14, U1.15, U1.2, U1.7, U2.10, U2.14, U2.15, U2.2, U2.7
- net MOTOR1: now also C14.1, U3.8, U3.9; no longer C9.1, U1.8, U1.9
- net MOTOR2: now also C14.2, U3.5, U3.6; no longer C9.2, U1.5, U1.6
- net MOTOR3: now also C15.1, U4.8, U4.9; no longer C10.1, U2.8, U2.9
- net MOTOR4: now also C15.2, U4.5, U4.6; no longer C10.2, U2.5, U2.6
- net SIG1: now also U1.20, U4.11; no longer JP1.4, U2.11
- net SIG2: now also U1.16, U4.12; no longer JP1.5, U2.12
- net SIG3: now also U1.28, U3.11; no longer JP1.6, U1.11
- net SIG4: now also U1.29, U3.12; no longer JP1.7, U1.12
- net V-ADC: now also R3.2, R4.1; no longer JP1.3, R1.1
Routing:
- net 3.3V: track 4.66 -> 51.1 mm, vias 0 -> 7
- net GND: track 7.15 -> 42.2 mm, vias 33 -> 59
- net RADIO-RST: track 0.00 -> 31.9 mm, vias 0 -> 4
- net RADIO-VDD: track 0.00 -> 22.8 mm, vias 0 -> 2
- net SLEEP: track 13.4 -> 0.00 mm, vias 2 -> 0
- net SIG2: track 9.41 -> 20.7 mm, vias 0 -> 2
- net SIG1: track 9.05 -> 18.3 mm, vias 0 -> 2
- net BATT-ADC: track 0.00 -> 6.98 mm, vias 0 -> 1
- net U0TXD: track 0.00 -> 6.65 mm
- net AUX1: track 0.00 -> 6.56 mm
- net ESP-EN: track 0.00 -> 6.52 mm
- net U0RXD: track 0.00 -> 5.80 mm
- net RADIO-BUSY: track 0.00 -> 5.77 mm, vias 0 -> 1
- net AUX2: track 0.00 -> 5.71 mm
- net RADIO-DIO: track 0.00 -> 5.47 mm, vias 0 -> 1
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- added copper zone on layer 15, net 3.3V
- added copper zone on layer 2, net GND
Other:
- board size 18 x 15 mm -> 18 x 27 mm
- board text added: "1"
- board text added: "19"
- board text added: "22"
- board text added: "3"
- board text added: "GND"
- board text added: "P1"
- board text added: "P2"
- board text added: "RX"
- board text added: "TX"
- board text removed: "G"

Commit message: second gen gerbers
Parts:
- R4: device shrew-common:0402-RES -> shrew-common:0402-REV
Routing:
- net GND: vias 59 -> 58
Other:
- board text added: "A"
- board text added: "B"
- board text added: "SHREW-MEGA"
Changed lines of the file:
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@@
 <layer number="21" name="tPlace" color="7" fill="1" visible="yes" active="yes"/>
 <layer number="22" name="bPlace" color="7" fill="1" visible="yes" active="yes"/>
-<layer number="23" name="tOrigins" color="15" fill="1" visible="yes" active="yes"/>
-<layer number="24" name="bOrigins" color="15" fill="1" visible="yes" active="yes"/>
+<layer number="23" name="tOrigins" color="15" fill="1" visible="no" active="yes"/>
+<layer number="24" name="bOrigins" color="15" fill="1" visible="no" active="yes"/>
 <layer number="25" name="tNames" color="7" fill="1" visible="no" active="yes"/>
 <layer number="26" name="bNames" color="7" fill="1" visible="no" active="yes"/>
@@
 <layer number="39" name="tKeepout" color="4" fill="11" visible="no" active="yes"/>
 <layer number="40" name="bKeepout" color="1" fill="11" visible="no" active="yes"/>
-<layer number="41" name="tRestrict" color="4" fill="10" visible="yes" active="yes"/>
-<layer number="42" name="bRestrict" color="1" fill="10" visible="yes" active="yes"/>
-<layer number="43" name="vRestrict" color="2" fill="10" visible="yes" active="yes"/>
+<layer number="41" name="tRestrict" color="4" fill="10" visible="no" active="yes"/>
+<layer number="42" name="bRestrict" color="1" fill="10" visible="no" active="yes"/>
+<layer number="43" name="vRestrict" color="2" fill="10" visible="no" active="yes"/>
 <layer number="44" name="Drills" color="7" fill="1" visible="no" active="yes"/>
 <layer number="45" name="Holes" color="7" fill="1" visible="no" active="yes"/>
@@
 <text x="2.5" y="21.8" size="1" layer="22" rot="MR180" align="center-left">1</text>
 <text x="2.5" y="19.1" size="1" layer="22" rot="MR180" align="center-left">3</text>
+<text x="17.1" y="14.2" size="1" layer="22" font="vector" ratio="10" rot="MR90" align="center-left">SHREW-MEGA</text>
+<text x="3.7" y="1.7" size="0.8" layer="22" font="vector" ratio="10" rot="MR0" align="center">A</text>
+<text x="3.9" y="1.7" size="0.8" layer="21" font="vector" ratio="10" align="center">A</text>
+<text x="14.3" y="1.6" size="0.8" layer="21" font="vector" ratio="10" align="center">B</text>
+<text x="14.1" y="1.6" size="0.8" layer="22" font="vector" ratio="10" rot="MR0" align="center">B</text>
 </plain>
 <attributes>
@@
 <attribute name="VALUE" x="11.503" y="10.104" size="0.4064" layer="28" rot="MR90"/>
 </element>
-<element name="R4" library="shrew-common" package="0402-RES" value="" x="2.9" y="12.4" smashed="yes" rot="MR0">
+<element name="R4" library="shrew-common" package="0402-REV" value="" x="2.9" y="12.4" smashed="yes" rot="MR0">
 <attribute name="NAME" x="3.789" y="13.0985" size="1.016" layer="26" font="vector" rot="MR0"/>
 <attribute name="VALUE" x="3.9795" y="11.257" size="0.4064" layer="28" rot="MR0"/>
@@
 <via x="16.18" y="18.77" extent="1-16" drill="0.3" shape="octagon"/>
 <polygon width="0.254" layer="2" spacing="0.1524" isolate="0.2032" thermals="no">
-<vertex x="1.5" y="2.9"/>
+<vertex x="1.5" y="3.8"/>
 <vertex x="1.5" y="27"/>
 <vertex x="18" y="27"/>
-<vertex x="18" y="2.9"/>
+<vertex x="18" y="3.8"/>
 </polygon>
 <via x="11.6" y="22.4" extent="1-16" drill="0.3" shape="octagon"/>
@@
 <via x="5.4" y="13.5" extent="1-16" drill="0.3" shape="octagon"/>
 <via x="3.8" y="14.8" extent="1-16" drill="0.3" shape="octagon"/>
-<via x="2" y="13.4" extent="1-16" drill="0.3" shape="octagon"/>
 <via x="3.8" y="13.4" extent="1-16" drill="0.3" shape="octagon"/>
 <contactref element="IC1" pad="2"/>
@@
 <wire x1="5.95" y1="17.25" x2="5.95" y2="17.1" width="0.254" layer="16"/>
 <polygon width="0.2032" layer="15" spacing="0.1524" isolate="0.2032" thermals="no">
-<vertex x="1.5" y="2.9"/>
+<vertex x="1.5" y="3.8"/>
 <vertex x="1.5" y="27"/>
 <vertex x="18" y="27"/>
-<vertex x="18" y="2.9"/>
+<vertex x="18" y="3.8"/>
 </polygon>
 <via x="12.4" y="16" extent="1-16" drill="0.3" shape="octagon"/>
@@
 <contactref element="R3" pad="2"/>
 <contactref element="R4" pad="1"/>
-<wire x1="10.5" y1="12.8" x2="3.95" y2="12.8" width="0.1524" layer="16"/>
-<wire x1="3.95" y1="12.8" x2="3.55" y2="12.4" width="0.1524" layer="16"/>
+<wire x1="10.5" y1="12.8" x2="3.8" y2="12.8" width="0.1524" layer="16"/>
 <wire x1="10.5" y1="12.8" x2="12.1" y2="14.4" width="0.1524" layer="16"/>
+<wire x1="3.8" y1="12.8" x2="3.4" y2="12.4" width="0.1524" layer="16"/>
 </signal>
 <signal name="N$5">
@@
 <wire x1="3.9" y1="9.6" x2="2" y2="9.6" width="0.6" layer="16"/>
 <wire x1="2" y1="9.6" x2="1.6" y2="10" width="0.6" layer="16"/>
-<wire x1="2.25" y1="12.4" x2="2.25" y2="10.65" width="0.4064" layer="16"/>
-<wire x1="2.25" y1="10.65" x2="1.6" y2="10" width="0.4064" layer="16"/>
+<wire x1="2.4" y1="10.8" x2="1.6" y2="10" width="0.4064" layer="16"/>
 <contactref element="C24" pad="1"/>
 <contactref element="IC1" pad="5"/>
 <contactref element="IC1" pad="4"/>
 <wire x1="8.5" y1="7.755" x2="8.5" y2="8.3" width="0.4064" layer="16"/>
-<wire x1="8.5" y1="8.3" x2="8" y2="8.3" width="0.4064" layer="16"/>
+<wire x1="8.5" y1="8.3" x2="7.55" y2="8.3" width="0.4064" layer="16"/>
 <wire x1="7.55" y1="8.3" x2="5" y2="8.3" width="0.4064" layer="16"/>
 <wire x1="5" y1="8.3" x2="4.4" y2="8.9" width="0.4064" layer="16"/>
@@
 <wire x1="4.4" y1="9.1" x2="3.9" y2="9.6" width="0.4064" layer="16"/>
 <wire x1="7.55" y1="7.755" x2="7.55" y2="8.3" width="0.4064" layer="16"/>
-<wire x1="7.55" y1="8.3" x2="8" y2="8.3" width="0.4064" layer="16"/>
+<wire x1="2.4" y1="10.8" x2="2.4" y2="12.4" width="0.4064" layer="16"/>
 </signal>
 <signal name="MOTOR2">
