File: electrical/shrew-pro.brd (EAGLE design)
At the start: 18 x 27 mm, 52 parts, among them IC1 LMR16006YQ3DDCTQ1, U1 ESP32-PICO-D4, U2 SX1280IMLTRT, U3 DRV8244SQRYJRQ1, U4 DRV8244SQRYJRQ1, X1 PIN-1X-BIG, X2 PIN-1X-BIG, X3 PIN-1X-BIG, X4 PIN-1X-BIG, X5 PIN-1X-BIG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

Commit message: placed a PCBA order for shrew-lite
Parts:
- C14, C15: value (none) -> 100n
- C16, C18, C19, C20, C21, C22, C23: value (none) -> 10u
- R4: value (none) -> 68K
Other:
- board text added: "SHREW-PRO"
- board text removed: "SHREW-MEGA"
Changed lines of the file:
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@@
 <text x="2.5" y="21.8" size="1" layer="22" rot="MR180" align="center-left">1</text>
 <text x="2.5" y="19.1" size="1" layer="22" rot="MR180" align="center-left">3</text>
-<text x="17.1" y="14.2" size="1" layer="22" font="vector" ratio="10" rot="MR90" align="center-left">SHREW-MEGA</text>
+<text x="17.1" y="14.2" size="1" layer="22" font="vector" ratio="10" rot="MR90" align="center-left">SHREW-PRO</text>
 <text x="3.7" y="1.7" size="0.8" layer="22" font="vector" ratio="10" rot="MR0" align="center">A</text>
 <text x="3.9" y="1.7" size="0.8" layer="21" font="vector" ratio="10" align="center">A</text>
@@
 <element name="X3" library="shrew-core" package="PAD-1X-BIG" value="PIN-1X-BIG" x="12" y="1.6" smashed="yes"/>
 <element name="X4" library="shrew-core" package="PAD-1X-BIG" value="PIN-1X-BIG" x="16.4" y="1.6" smashed="yes"/>
-<element name="C14" library="shrew-common" package="0402-CAP" value="" x="3.8" y="3.39" smashed="yes" rot="R180">
+<element name="C14" library="shrew-common" package="0402-CAP" value="100n" x="3.8" y="3.39" smashed="yes" rot="R180">
 <attribute name="NAME" x="5.011" y="3.1085" size="1.016" layer="25" font="vector"/>
 <attribute name="VALUE" x="4.8795" y="4.533" size="0.4064" layer="27" rot="R180"/>
 </element>
-<element name="C15" library="shrew-common" package="0402-CAP" value="" x="14.2" y="3.39" smashed="yes" rot="R180">
+<element name="C15" library="shrew-common" package="0402-CAP" value="100n" x="14.2" y="3.39" smashed="yes" rot="R180">
 <attribute name="NAME" x="15.411" y="3.2085" size="1.016" layer="25" font="vector"/>
 <attribute name="VALUE" x="15.2795" y="4.533" size="0.4064" layer="27" rot="R180"/>
@@
 <element name="X5" library="shrew-core" package="PAD-1X-BIG" value="PIN-1X-BIG" x="1.6" y="10" smashed="yes"/>
 <element name="X6" library="shrew-core" package="PAD-1X-BIG" value="PIN-1X-BIG" x="16.4" y="10" smashed="yes"/>
-<element name="C16" library="shrew-common" package="0805" value="" x="1.7" y="4.3" smashed="yes" rot="MR180">
+<element name="C16" library="shrew-common" package="0805" value="10u" x="1.7" y="4.3" smashed="yes" rot="MR180">
 <attribute name="NAME" x="3.238" y="4.7745" size="1.016" layer="26" font="vector" rot="MR180"/>
 <attribute name="VALUE" x="0.684" y="5.697" size="0.4064" layer="28" rot="MR180"/>
 </element>
-<element name="C18" library="shrew-common" package="0805" value="" x="1.7" y="5.9" smashed="yes" rot="MR180">
+<element name="C18" library="shrew-common" package="0805" value="10u" x="1.7" y="5.9" smashed="yes" rot="MR180">
 <attribute name="NAME" x="3.238" y="6.3745" size="1.016" layer="26" font="vector" rot="MR180"/>
 <attribute name="VALUE" x="0.684" y="7.297" size="0.4064" layer="28" rot="MR180"/>
 </element>
-<element name="C19" library="shrew-common" package="0805" value="" x="1.7" y="7.5" smashed="yes" rot="MR180">
+<element name="C19" library="shrew-common" package="0805" value="10u" x="1.7" y="7.5" smashed="yes" rot="MR180">
 <attribute name="NAME" x="3.138" y="7.9745" size="1.016" layer="26" font="vector" rot="MR180"/>
 <attribute name="VALUE" x="0.684" y="8.897" size="0.4064" layer="28" rot="MR180"/>
 </element>
-<element name="C20" library="shrew-common" package="0805" value="" x="3.9" y="8.7" smashed="yes" rot="MR270">
+<element name="C20" library="shrew-common" package="0805" value="10u" x="3.9" y="8.7" smashed="yes" rot="MR270">
 <attribute name="NAME" x="3.0745" y="9.462" size="1.016" layer="26" font="vector" rot="MR270"/>
 <attribute name="VALUE" x="5.297" y="9.716" size="0.4064" layer="28" rot="MR270"/>
@@
 <attribute name="VALUE" x="11.503" y="10.104" size="0.4064" layer="28" rot="MR90"/>
 </element>
-<element name="R4" library="shrew-common" package="0402-REV" value="" x="2.9" y="12.4" smashed="yes" rot="MR0">
+<element name="R4" library="shrew-common" package="0402-REV" value="68K" x="2.9" y="12.4" smashed="yes" rot="MR0">
 <attribute name="NAME" x="3.789" y="13.0985" size="1.016" layer="26" font="vector" rot="MR0"/>
 <attribute name="VALUE" x="3.9795" y="11.257" size="0.4064" layer="28" rot="MR0"/>
@@
 <attribute name="NAME" x="9.4234" y="6.865" size="1.016" layer="27" font="vector" ratio="6" rot="SR0"/>
 </element>
-<element name="C21" library="shrew-common" package="0805" value="" x="16.4" y="7.15" smashed="yes" rot="MR180">
+<element name="C21" library="shrew-common" package="0805" value="10u" x="16.4" y="7.15" smashed="yes" rot="MR180">
 <attribute name="NAME" x="15.638" y="6.3245" size="1.016" layer="26" font="vector" rot="MR180"/>
 <attribute name="VALUE" x="15.384" y="8.547" size="0.4064" layer="28" rot="MR180"/>
 </element>
-<element name="C22" library="shrew-common" package="0805" value="" x="16.4" y="5.55" smashed="yes" rot="MR180">
+<element name="C22" library="shrew-common" package="0805" value="10u" x="16.4" y="5.55" smashed="yes" rot="MR180">
 <attribute name="NAME" x="15.638" y="4.7245" size="1.016" layer="26" font="vector" rot="MR180"/>
 <attribute name="VALUE" x="15.384" y="6.947" size="0.4064" layer="28" rot="MR180"/>
 </element>
-<element name="C23" library="shrew-common" package="0805" value="" x="16.4" y="3.95" smashed="yes" rot="MR180">
+<element name="C23" library="shrew-common" package="0805" value="10u" x="16.4" y="3.95" smashed="yes" rot="MR180">
 <attribute name="NAME" x="15.638" y="3.1245" size="1.016" layer="26" font="vector" rot="MR180"/>
 <attribute name="VALUE" x="15.384" y="5.347" size="0.4064" layer="28" rot="MR180"/>

Commit message: wip
Parts:
- added TP1, TP2, TP3: (no value), shrew-common:1X01-1.0MM-TP
Connections:
- net RADIO-RST: now also TP3.1
- net SIG1: now also TP1.1
- net SIG2: now also TP2.1
Routing:
- net GND: track 42.2 -> 46.4 mm, vias 58 -> 63
- net SIG1: track 18.3 -> 19.1 mm
- net SIG2: track 20.7 -> 21.3 mm
- net RADIO-RST: track 31.9 -> 32.4 mm
- net +24V: vias 1 -> 2
- added copper zone on layer 15, net +24V
- added copper zone on layer 15, net GND
Other:
- board text removed: "V"
