File: electrical/shrew-lite.sch (EAGLE design)
At the start: 47 parts, among them IC1 Vreg +3V3, U1 ESP32-PICO-D4, U2 SX1280IMLTRT, U3 DRV8231DSGR, U4 DRV8231DSGR, X1 PIN-1X-BIG, X2 PIN-1X-BIG, X3 PIN-1X-BIG, X4 PIN-1X-BIG, X5 PIN-1X-MED, X6 PIN-1X-MED, X7 PIN-1X-MED, X8 PIN-1X-MED, Y1 52MHz TCXO

Commit message: placed a PCBA order for shrew-lite
Parts:
- C11: value 10uF 25V -> 10u
- C14, C15: value (none) -> 100n
- C16, C18, C19, C20, C21: value (none) -> 10u
- R4: value (none) -> 68K
Connections:
- net V-ADC renamed N$4
Other:
- note removed: "not actually +24V"
- moved on the sheet: C17, D1, EDGE1, JP1, R2, R3, R4

Commit message: sorted component ref des
Parts:
- removed EDGE1: (no value), shrew-common:M05PTH
- removed FL1: 2450FM07D0034T, shrew-core:2450FM07D0034T
- added JP2: (no value), shrew-common:M07-2MM-TH-TINY
- added Y2: 52MHz TCXO, shrew-common:OSCILLATOR-TG2016SMN
- C1: value 1n -> 10u; device shrew-common:CAP0402-REV -> shrew-common:CAP0805
- C10: value 100n -> 470n
- C11: value 10u -> DNP; device shrew-common:CAP0805 -> shrew-common:CAP0402-CAP
- C12: value DNP -> 470n; device shrew-common:CAP0402-CAP -> shrew-common:CAP0402-REV
- C13: value 470n -> 10n
- C14: value 100n -> 10n; device shrew-common:CAP0402-CAP -> shrew-common:CAP0402-REV
- C15: value 100n -> 1n; device shrew-common:CAP0402-CAP -> shrew-common:CAP0402-REV
- C16, C18: value 10u -> 100n; device shrew-common:CAP0805 -> shrew-common:CAP0402-REV
- C17: value 470n -> 100n
- C19: value 10u -> 470n; device shrew-common:CAP0805 -> shrew-common:CAP0402-REV
- C2: value 470n -> 10u; device shrew-common:CAP0402-REV -> shrew-common:CAP0805
- C20, C21: value 10u -> 100n; device shrew-common:CAP0805 -> shrew-common:CAP0402-CAP
- C3, C4: value 10n -> 10u; device shrew-common:CAP0402-REV -> shrew-common:CAP0805
- C5, C9: value 100n -> 10u; device shrew-common:CAP0402-REV -> shrew-common:CAP0805
- JP1: device shrew-common:M07-2MM-TH-TINY -> shrew-common:M05PTH
- R2: value 10K -> 68K; device shrew-common:RESISTOR0402-REV -> shrew-common:RESISTOR0402-RES
- R4: value 68K -> 10K; device shrew-common:RESISTOR0402-RES -> shrew-common:RESISTOR0402-REV
- X1, X2, X3, X4: value PIN-1X-BIG -> PIN-1X-MED; device shrew-core:PIN-1X-BIG -> shrew-core:PIN-1X-MED
- X5, X6, X7, X8: value PIN-1X-MED -> PIN-1X-BIG; device shrew-core:PIN-1X-MED -> shrew-core:PIN-1X-BIG
- Y1: value 52MHz TCXO -> 2450FM07D0034T; device shrew-common:OSCILLATOR-TG2016SMN -> shrew-core:2450FM07D0034T
Connections:
- net +24V: now also C2.1, C3.1, C4.1, C5.1, R2.2, X1.P$1, X2.P$1; no longer C16.1, C18.1, C19.1, C20.1, R4.2, X5.P$1, X7.P$1
- net 3.3V: now also C1.1, C16.2, C17.2, C18.2, C6.1, C7.1, JP2.2, Y2.VCC; no longer C10.1, C11.1, C21.1, C5.2, C6.2, C7.2, JP1.2, Y1.VCC
- net AUX1: now also JP1.1; no longer EDGE1.1
- net AUX2: now also JP1.2; no longer EDGE1.2
- net BATT-ADC: now also C12.1, R4.2; no longer C17.1, R2.2
- net ESP-BOOT: now also C11.2; no longer C12.2
- net ESP-EN: now also C10.2; no longer C13.2
- net GND: now also C1.2, C10.1, C11.1, C12.2, C14.1, C16.1, C17.1, C18.1, C19.1, C2.2, C3.2, C4.2, C5.2, C6.2, C7.2, JP1.5, JP2.1, R4.1, X3.P$1, X4.P$1, Y2.GND; no longer C10.2, C11.2, C12.1, C16.2, C17.2, C18.2, C19.2, C2.1, C20.2, C21.2, C3.1, C4.1, C5.1, C6.1, C7.1, EDGE1.5, JP1.1, R2.1, X6.P$1, X8.P$1, Y1.GND
- net MOTOR1: now also C21.2, X8.P$1; no longer C15.2, X3.P$1
- net MOTOR2: now also C21.1, X6.P$1; no longer C15.1, X4.P$1
- net MOTOR3: now also C20.2, X7.P$1; no longer C14.2, X1.P$1
- net MOTOR4: now also C20.1, X5.P$1; no longer C14.1, X2.P$1
- net N$11: now also C14.2; no longer C3.2
- net N$2: now also C15.1, Y2.OUT; no longer C1.1, Y1.OUT
- net N$3: now also C15.2; no longer C1.2
- net N$4: now also JP2.3, R2.1; no longer JP1.3, R4.1
- net N$6: now also Y1.IN; no longer FL1.IN
- net N$7: now also Y1.OUT; no longer FL1.OUT
- net RADIO-VDD: now also C13.2, C19.2; no longer C2.2, C4.2
- net SIG1: now also JP2.4; no longer JP1.4
- net SIG2: now also JP2.5; no longer JP1.5
- net SIG3: now also JP2.6; no longer JP1.6
- net SIG4: now also JP2.7; no longer JP1.7
- net U0RXD: now also JP1.3; no longer EDGE1.3
- net U0TXD: now also JP1.4; no longer EDGE1.4
Other:
- moved on the sheet: ANT2, C1, C10, C12, C13, C14, C15, C16, C17, C18, C19, C2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

Commit message: shrew pro prototype sent off to manufacturing
Parts:
- removed JP2: (no value), shrew-common:M07-2MM-TH-TINY
- R2: device shrew-common:RESISTOR0402-RES -> shrew-common:RESISTOR0402-REV
Connections:
- net 3.3V: no longer JP2.2
- net GND: no longer JP2.1
- net N$4: no longer JP2.3
- net SIG1: no longer JP2.4
- net SIG2: no longer JP2.5
- net SIG3: no longer JP2.6
- net SIG4: no longer JP2.7

Commit message: shrew-lite new buck vreg
Parts:
- removed D1: 3V6, shrew-common:DIODE-ZENER-BZT52
- added C22, C23: 100n, shrew-common:CAP0402-CAP
- added L2: 15u, shrew-common:INDUCTOR0805
- C1, C9: value 10u -> 100n; device shrew-common:CAP0805 -> shrew-common:CAP0402-REV
- C10, C19: value 470n -> 100n
- C11: value DNP -> 10u; device shrew-common:CAP0402-CAP -> shrew-common:CAP0805
- C13: value 10n -> DNP; device shrew-common:CAP0402-REV -> shrew-common:CAP0402-CAP
- C14: value 10n -> 470n
- C15: value 1n -> 10n
- C16: value 100n -> 10n
- C17: value 100n -> 1n
- C2, C3: value 10u -> 22u
- C20: device shrew-common:CAP0402-CAP -> shrew-common:CAP0402-REV
- C21: value 100n -> 470n; device shrew-common:CAP0402-CAP -> shrew-common:CAP0402-REV
- C6, C7: value 100n -> 10u; device shrew-common:CAP0402-REV -> shrew-common:CAP0805
- IC1: value Vreg +3V3 -> AP63203WU; device shrew-common:V_REG_SOT89-SOT89 -> shrew-core:AP63203WU
- L1: value 15u -> 10u
Connections:
- new net N$10: C1.2, IC1.SW, L1.1
- new net N$12: C1.1, IC1.BST
- net +24V: now also C6.1, C7.1, IC1.EN, IC1.VIN; no longer C2.1, C3.1, IC1.IN
- net 3.3V: now also C10.1, C11.1, C19.2, C2.1, C20.2, C3.1, IC1.FB, L1.2; no longer C1.1, C16.2, C17.2, C6.1, C7.1, IC1.VO
- net BATT-ADC: now also C14.1; no longer C12.1, D1.C
- net ESP-BOOT: now also C13.2; no longer C11.2
- net ESP-EN: now also C12.2; no longer C10.2
- net GND: now also C10.2, C11.2, C12.1, C14.2, C15.1, C20.1, C21.1; no longer C1.2, C10.1, C11.1, C12.2, C14.1, C17.1, D1.A, IC1.TAB
- net MOTOR1: now also C23.2; no longer C21.2
- net MOTOR2: now also C23.1; no longer C21.1
- net MOTOR3: now also C22.2; no longer C20.2
- net MOTOR4: now also C22.1; no longer C20.1
- net N$11: now also C16.2; no longer C14.2
- net N$2: now also C17.1; no longer C15.1
- net N$3: now also C17.2; no longer C15.2
- net N$9: now also L2.2; no longer L1.2
- net RADIO-VDD: now also C15.2, C21.2, L2.1; no longer C13.2, C19.2, L1.1
Other:
- moved on the sheet: ANT2, C1, C10, C12, C14, C15, C16, C17, C18, C19, C2, C20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

Commit message: shrew-lite buck vreg wip, shorter
Parts:
- added C24, C25, C26: 10u, shrew-common:CAP0402-REV
- added JP2: M01-1.0MM-TP, shrew-common:M01-1.0MM-TP
- C11: device shrew-common:CAP0805 -> shrew-common:CAP0402-REV
- C2, C3: value 22u -> 10u; device shrew-common:CAP0805 -> shrew-common:CAP0402-REV
Connections:
- net 3.3V: now also C24.1, C25.1, C26.1, JP2.1
- net GND: now also C24.2, C25.2, C26.2
Other:
- moved on the sheet: C1, C2, C3, C4, C5, C6, C7, IC1, L1

Commit message: shrew-lite another prototype order
Parts:
- C10, C8, C9: value 100n -> 10u; device shrew-common:CAP0402-REV -> shrew-common:CAP0805
- C11: value 10u -> 100n
- C12, C21: value 470n -> 100n
- C13: value DNP -> 100n; device shrew-common:CAP0402-CAP -> shrew-common:CAP0402-REV
- C14: value 470n -> 10u
- C15: value 10n -> 470n
- C16: value 10n -> DNP; device shrew-common:CAP0402-REV -> shrew-common:CAP0402-CAP
- C17: value 1n -> 470n
- C18, C19: value 100n -> 10n
- C20: value 100n -> 1n
- C22, C23: device shrew-common:CAP0402-CAP -> shrew-common:CAP0402-REV
- C24: value 10u -> 470n
- C25, C26: value 10u -> 100n; device shrew-common:CAP0402-REV -> shrew-common:CAP0402-CAP
- C4, C5, C6: device shrew-common:CAP0805 -> shrew-common:CAP0402-REV
- JP1: value (none) -> M01-1.0MM-TP; device shrew-common:M05PTH -> shrew-common:M01-1.0MM-TP
- JP2: value M01-1.0MM-TP -> (none); device shrew-common:M01-1.0MM-TP -> shrew-common:M05PTH
- L1: value 10u -> 10uH
Connections:
- net +24V: now also C10.1, C8.1, C9.1; no longer C4.1, C5.1, C6.1
- net 3.3V: now also C12.1, C13.1, C14.1, C21.2, C22.2, C23.2, C4.1, C5.1, C6.1, JP1.1; no longer C10.1, C18.2, C19.2, C20.2, C24.1, C25.1, C26.1, C8.1, C9.1, JP2.1
- net AUX1: now also JP2.1; no longer JP1.1
- net AUX2: now also JP2.2; no longer JP1.2
- net BATT-ADC: now also C17.1; no longer C14.1
- net ESP-BOOT: now also C16.2; no longer C13.2
- net ESP-EN: now also C15.2; no longer C12.2
- net GND: now also C12.2, C13.2, C17.2, C22.1, C23.1, C24.1, JP2.5; no longer C12.1, C13.1, C20.1, C24.2, C25.2, C26.2, JP1.5
- net MOTOR1: now also C26.2; no longer C23.2
- net MOTOR2: now also C26.1; no longer C23.1
- net MOTOR3: now also C25.2; no longer C22.2
- net MOTOR4: now also C25.1; no longer C22.1
- net N$11: now also C19.2; no longer C16.2
- net N$2: now also C20.1; no longer C17.1
- net N$3: now also C20.2; no longer C17.2
- net RADIO-VDD: now also C18.2, C24.2; no longer C15.2, C21.2
- net U0RXD: now also JP2.3; no longer JP1.3
- net U0TXD: now also JP2.4; no longer JP1.4
Other:
- moved on the sheet: ANT2, C10, C11, C12, C14, C15, C17, C18, C19, C20, C21, C22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
