File: electrical/shrew-lite.sch (EAGLE design)
At the start: 52 parts, among them IC1 AP63203WU, U1 ESP32-PICO-D4, U2 SX1280IMLTRT, U3 DRV8231DSGR, U4 DRV8231DSGR, X1 PIN-1X-MED, X2 PIN-1X-MED, X3 PIN-1X-MED, X4 PIN-1X-MED, X5 PIN-1X-BIG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

Commit message: PCB changes for better EMI emissions
Parts:
- added C27, C28, C29: 100n, shrew-common:CAP0402-REV
- added C30: 0.5pF, shrew-common:CAP0402-REV
- ANT1, ANT2: value 74889302450 -> ANT3216LL00R2400A
Connections:
- net 3.3V: now also C27.1, C28.1, C29.1
- net GND: now also C27.2, C28.2, C29.2, C30.2
- net N$1: now also C30.1
Other:
- moved on the sheet: ANT2, C11, C12, C13, C14, C18, C19, C20, C21, C22, C23, C24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
