File: electrical/shrew-lite.sch (EAGLE design)
At the start: 52 parts, among them IC1 AP63203WU, U1 ESP32-PICO-D4, U2 SX1280IMLTRT, U3 DRV8231DSGR, U4 DRV8231DSGR, X1 PIN-1X-MED, X2 PIN-1X-MED, X3 PIN-1X-MED, X4 PIN-1X-MED, X5 PIN-1X-BIG, X6 PIN-1X-BIG, X7 PIN-1X-BIG, X8 PIN-1X-BIG, Y1 2450FM07D0034T, Y2 52MHz TCXO

Commit message: shrew lite mfg files update
Parts:
- ANT1: value 74889302450 -> 2.4G / 1206; JLC_ROTATION (none) -> 180; LCSC (none) -> C127620
- ANT2: value 74889302450 -> 2.4G / 1206; LCSC (none) -> C127620
- C1, C11, C12, C13, C21, C22, C23, C25, C26: LCSC (none) -> C1581
- C14, C2, C3, C4, C5, C6: LCSC (none) -> C15525
- C15: LCSC (none) -> C7393859
- C16, JP1, JP2, X1, X2, X3, X4, X5, X6, X7, X8: DNP (none) -> 1
- C18, C19: LCSC (none) -> C15195
- C20: LCSC (none) -> C1523
- IC1: JLC_ROTATION (none) -> 180
- L2: LCSC (none) -> C6364731
- R1, R3, R4: LCSC (none) -> C25744
- R2: LCSC (none) -> C2909379
- U1, U2: JLC_ROTATION (none) -> -90
- U3, U4: JLC_ROTATION (none) -> 90
- Y1: value 2450FM07D0034T -> 2450FM07D0034001T; LCSC (none) -> C6054595
- Y2: JLC_ROTATION (none) -> -90; LCSC (none) -> C22434896
