File: electrical/shrew-programmer.sch (EAGLE design)
At the start: 9 parts, among them SW1 SWITCH-ROCKER-3PIN-2MNT, X1 PROG-JIG

Commit message: another programmer PCB
Parts:
- removed JP2: (no value), shrew-common:M02PTH
- added JMP1, JMP2: JUMPER-3PTH, shrew-common:JUMPER-3PTH
- added JMP3: (no value), shrew-common:JUMPER-2PTH
- added JP3: (no value), shrew-common:M023.5MM
- added R2, R3: (no value), shrew-common:RESISTOR0603-RES
- added X2: PROG-JIG-PRO, shrew-core:PROG-JIG-PRO
- added X3: PROG-JIG-ZERO, shrew-core:PROG-JIG-ZERO
- LED1: device shrew-common:LED5MM -> shrew-common:LED1206
- X1: value PROG-JIG -> PROG-JIG-LITE; device shrew-core:PROG-JIG -> shrew-core:PROG-JIG-LITE
Connections:
- removed net N$3: JP1.3, X1.RX1, X1.RX2
- new net 3V3: JMP2.3, X1.3V3, X2.3V3
- new net BOOT: JMP3.1, X1.BOOT, X2.BOOT, X3.BOOT
- new net PC-RX: R3.1, X1.TX, X2.TX, X3.TX
- new net PC-TX: R2.1, X1.RX, X2.RX, X3.RX
- new net V-DC: JMP1.1, JP3.2
- new net V-USB: JMP1.3, JP1.4
- new net VBAT: JMP2.1, X1.VBAT, X2.VBAT, X2.VBAT2, X3.VBAT, X3.VBAT2
- net GND: now also JMP3.2, JP3.1, X1.G1, X1.GND, X2.G1, X2.GND, X3.G1, X3.G2, X3.GND; no longer JP2.1, X1.GND1, X1.GND2
- net N$1: now also JP1.3, R2.2; no longer JP1.2, X1.TX1, X1.TX2
- net N$2: now also JP1.2, R3.2; no longer LED1.A, SW1.1, X1.PWR1, X1.PWR2
- net N$4: now also JMP1.2; no longer JP1.4
- net N$6: now also JMP2.2, LED1.A, SW1.1; no longer JP2.2, X1.BOOT1, X1.BOOT2
Other:
- moved on the sheet: C1, C2, C3
