File: electrical/shrew-pro.sch (EAGLE design)
At the start: 58 parts, among them IC1 LMR16006YQ3DDCTQ1, U1 ESP32-PICO-D4, U2 SX1280IMLTRT, U3 DRV8244HQRYJRQ1, U4 DRV8244HQRYJRQ1, X1 PIN-1X-BIG, X2 PIN-1X-BIG, X3 PIN-1X-BIG, X4 PIN-1X-BIG, X5 PIN-1X-BIG, X6 PIN-1X-BIG, Y1 2450FM07D0034T, Y2 52MHz TCXO

Commit message: PCB changes for better EMI emissions
Parts:
- added C32: DNP, shrew-common:CAP0402-CAP
- ANT1, ANT2: value 74889302450 -> ANT3216LL00R2400A
- C12: value 100n -> 10u; device shrew-common:CAP0402-REV -> shrew-common:CAP0805
- C15: value 10uF 25V -> 100n; device shrew-common:CAP0805 -> shrew-common:CAP0402-REV
- C16, C18: value 470n -> 100n
- C17: value DNP -> 100n; device shrew-common:CAP0402-CAP -> shrew-common:CAP0402-REV
- C19: value 10n -> 10uF 25V; device shrew-common:CAP0402-REV -> shrew-common:CAP0805
- C21: value 1n -> 10n
- C22: value 100n -> 1n
- C23: value 100n -> 470n
- C25: value 470n -> 0.5pF; device shrew-common:CAP0402-REV -> shrew-common:CAP0402-CAP
- C26, C27: device shrew-common:CAP0402-CAP -> shrew-common:CAP0402-REV
- C28: value 100nF -> 470n; device shrew-common:CAP0402-CAP -> shrew-common:CAP0402-REV
- C29: value 100nF -> 100n
- C3: value 10u -> 100n; device shrew-common:CAP0805 -> shrew-common:CAP0402-REV
- C30: value 100nF -> 100n; device shrew-common:CAP0402-REV -> shrew-common:CAP0402-CAP
- C31: value 0.5pF -> 470n; device shrew-common:CAP0402-CAP -> shrew-common:CAP0402-REV
- U1: value ESP32-PICO-D4 -> SX1280IMLTRT; device shrew-core:ESP32-PICO-D4 -> shrew-core:SX1280IMLTRT
- U2: value SX1280IMLTRT -> ESP32-PICO-D4; device shrew-core:SX1280IMLTRT -> shrew-core:ESP32-PICO-D4
Connections:
- net +24V: now also C12.1, C3.2, C4.1; no longer C3.1, C30.2, C5.1
- net 3.3V: now also C13.2, C14.2, C15.2, C16.1, C17.1, C18.1, C19.1, C26.2, C27.2, C5.1, U1.VBAT, U1.VBAT_IO, U2.VDD3P3_CPU, U2.VDD3P3_RTC, U2.VDDA, U2.VDDA3P3, U2.VDD_SDIO; no longer C12.1, C13.1, C14.1, C15.1, C22.2, C23.2, C28.2, C29.2, C4.1, U1.VDD3P3_CPU, U1.VDD3P3_RTC, U1.VDDA, U1.VDDA3P3, U1.VDD_SDIO, U2.VBAT, U2.VBAT_IO
- net AUX1: now also U2.IO19; no longer U1.IO19
- net AUX2: now also U2.IO22; no longer U1.IO22
- net BATT-ADC: now also C31.1, U2.IO4; no longer C18.1, U1.IO4
- net ESP-BOOT: now also C32.2, U2.IO0(BOOT); no longer C17.2, U1.IO0(BOOT)
- net ESP-EN: now also C23.2, U2.EN; no longer C16.2, U1.EN
- net GND: now also C13.1, C14.1, C15.1, C16.2, C17.2, C19.2, C21.1, C25.2, C26.1, C27.1, C3.1, C32.1, U1.GND_2, U1.GND_3, U1.GND_4, U1.GND_5, U1.GND_6, U1.GND_7, U2.IO15/MTDO; no longer C13.2, C14.2, C15.2, C16.1, C17.1, C19.1, C22.1, C25.1, C29.1, C3.2, C30.1, U1.IO15/MTDO, U2.GND_2, U2.GND_3, U2.GND_4, U2.GND_5, U2.GND_6, U2.GND_7
- net MOTOR1: now also C29.1; no longer C26.1
- net MOTOR2: now also C29.2; no longer C26.2
- net MOTOR3: now also C30.1; no longer C27.1
- net MOTOR4: now also C30.2; no longer C27.2
- net N$1: now also C25.1, U2.LNA_IN; no longer C31.1, U1.LNA_IN
- net N$11: now also C21.2, U1.VR_PA; no longer C20.2, U2.VR_PA
- net N$2: now also C22.1; no longer C21.1
- net N$3: now also C22.2, U1.XTA; no longer C21.2, U2.XTA
- net N$5: now also U2.IO14; no longer U1.IO14
- net N$6: now also U1.RFIO; no longer U2.RFIO
- net N$8: now also U2.IO2; no longer U1.IO2
- net N$9: now also U1.DCC_SW; no longer U2.DCC_SW
- net RADIO-BUSY: now also U1.BUSY, U2.IO23; no longer U1.IO23, U2.BUSY
- net RADIO-CS: now also U1.NSS_CTS, U2.IO32; no longer U1.IO32, U2.NSS_CTS
- net RADIO-DIO: now also U1.DIO1, U2.IO18; no longer U1.IO18, U2.DIO1
- net RADIO-RST: now also U1.NRESET, U2.IO21; no longer U1.IO21, U2.NRESET
- net RADIO-VDD: now also C20.2, C28.2, U1.DCC_FB, U1.VDD_INN; no longer C19.2, C25.2, U2.DCC_FB, U2.VDD_INN
- net RGBLED: now also U2.IO5; no longer U1.IO5
- net SIG1: now also U2.IO13; no longer U1.IO13
- net SIG2: now also U2.IO27; no longer U1.IO27
- net SIG3: now also U2.SD2/IO9; no longer U1.SD2/IO9
- net SIG4: now also U2.SD3/IO10; no longer U1.SD3/IO10
- net SPI-MISO: now also U1.MISO_TX, U2.IO26; no longer U1.IO26, U2.MISO_TX
- net SPI-MOSI: now also U1.MOSI_RX, U2.IO25; no longer U1.IO25, U2.MOSI_RX
- net SPI-SCK: now also U1.SCK_RTSN, U2.IO33; no longer U1.IO33, U2.SCK_RTSN
- net U0RXD: now also U2.U0RXD(IO3); no longer U1.U0RXD(IO3)
- net U0TXD: now also U2.U0TXD(IO1); no longer U1.U0TXD(IO1)
Other:
- moved on the sheet: ANT2, C10, C11, C12, C13, C14, C15, C16, C17, C18, C19, C20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
