File: electrical/shrew-lite.brd (EAGLE design)
At the start: 15.5 x 23 mm, 52 parts, among them IC1 AP63203WU, U1 ESP32-PICO-D4, U2 SX1280IMLTRT, U3 DRV8231DSGR, U4 DRV8231DSGR, X1 PIN-1X-MED, X2 PIN-1X-MED, X3 PIN-1X-MED, X4 PIN-1X-MED, X5 PIN-1X-BIG, X6 PIN-1X-BIG, X7 PIN-1X-BIG, X8 PIN-1X-BIG, Y1 2450FM07D0034T, Y2 52MHz TCXO

Commit message: shrew lite mfg files update
Parts:
- ANT1, ANT2: value 74889302450 -> 2.4G / 1206
- Y1: value 2450FM07D0034T -> 2450FM07D0034001T
